File: prj-kicad/pmod-wifi-esp32.kicad_pcb (KiCad board)
At the start: 4 copper layers, 38.1 x 20.3 mm, 28 parts, among them P1 PMOD, U1 ESP32, U2 M25P16-VME, X1 40MHz

Commit message: = UPD: Fix bug of flash memory ios ; add a signal to control "boot" pin from pmod
Connections:
- P1 pad 9: Net-(P1-Pad9) -> PMOD_BOOT
- U1 pad 23: Net-(U1-Pad23) -> PMOD_BOOT
- U1 pad 28: FL_D2 -> FL_SHD
- U1 pad 29: FL_D3 -> FL_SWP
- U1 pad 32: FL_D0 -> FL_SDO
- U1 pad 33: FL_D1 -> FL_SDI
- U2 pad 2: FL_D1 -> FL_SDO
- U2 pad 3: FL_D2 -> FL_SWP
- U2 pad 5: FL_D0 -> FL_SDI
- U2 pad 7: FL_D3 -> FL_SHD
Routing:
- net PMOD_BOOT: track 0.00 -> 25.3 mm, vias 0 -> 3
- net GND: track 124.0 -> 141.4 mm, vias 18 -> 22
- net FL_D0: track 16.5 -> 0.00 mm, vias 2 -> 0
- net FL_SDI: track 0.00 -> 16.5 mm, vias 0 -> 2
- net FL_SHD: track 0.00 -> 16.5 mm, vias 0 -> 2
- net FL_SDO: track 0.00 -> 16.5 mm, vias 0 -> 2
- net FL_SWP: track 0.00 -> 16.5 mm
- net FL_D3: track 12.7 -> 0.00 mm, vias 2 -> 0
- net FL_D1: track 11.9 -> 0.00 mm, vias 2 -> 0
- net FL_D2: track 9.53 -> 0.00 mm
- net FL_SCS: track 8.37 -> 13.9 mm
- net FL_SCK: track 13.6 -> 16.5 mm
Other:
- board text added: "PMOD-ESP32 rev2"
- board text removed: "JLCJLCJLCJLC"
- board text removed: "PMOD-ESP32 rev1"
