File: prj-kicad/pmod-wifi-esp32.sch (KiCad schematic (older format))
At the start: 24 parts, among them P1 PMOD, U1 ESP32, U2 M25P16-VME, X1 40MHz

Commit message: = ADD: PCB routing
Parts:
- added C12: 100nF, pmod-wifi-esp32:SMD0603, symbol pmod-wifi-esp32:C
- added FB1: FB120, pmod-wifi-esp32:SMD0603, symbol pmod-wifi-esp32:INDUCTOR
- A1: footprint (none) -> pmod-wifi-esp32:ANT_7488910245
- C1: footprint (none) -> pmod-wifi-esp32:SMD0805
- C10, C11, C2, C3, C4, C5, C6, C7, C8, C9, L1, L2, R1, R2: footprint (none) -> pmod-wifi-esp32:SMD0603
- TP1, TP2, TP3, TP4: footprint (none) -> pmod-wifi-esp32:TP_SMD
- U1: footprint (none) -> pmod-wifi-esp32:QFN48-04
- U2: footprint (none) -> pmod-wifi-esp32:SOIC-8
- X1: footprint (none) -> pmod-wifi-esp32:Q_3.2x2.5
Connections:
- net +3.3V: now also C12.1, FB1.2
- net GND: now also C12.2
- net VCC: now also FB1.1
Changed lines of the file:
@@
 F 0 "U1" H 8200 3850 60  0000 L CNN
 F 1 "ESP32" H 7300 2850 60  0000 R CNN
-F 2 "" H 7750 3500 60  0001 C CNN
+F 2 "pmod-wifi-esp32:QFN48-04" H 7750 3500 60  0001 C CNN
 F 3 "" H 7750 3500 60  0000 C CNN
 	1    7750 3350
@@
 F 0 "C2" H 8450 4750 50  0000 R CNN
 F 1 "10nF" H 8450 4550 50  0000 R CNN
-F 2 "" H 8500 4650 60  0001 C CNN
+F 2 "pmod-wifi-esp32:SMD0603" H 8500 4650 60  0001 C CNN
 F 3 "" H 8500 4650 60  0000 C CNN
 	1    8500 4650
@@
 F 0 "X1" H 7750 4612 60  0000 C CNN
 F 1 "40MHz" H 7750 4521 40  0000 C CNN
-F 2 "" H 7750 4350 60  0001 C CNN
+F 2 "pmod-wifi-esp32:Q_3.2x2.5" H 7750 4350 60  0001 C CNN
 F 3 "" H 7750 4350 60  0000 C CNN
 	1    7750 4350
@@
 F 0 "C3" H 9150 4750 50  0000 L CNN
 F 1 "3,3nF" H 9150 4550 50  0000 L CNN
-F 2 "" H 9100 4650 60  0001 C CNN
+F 2 "pmod-wifi-esp32:SMD0603" H 9100 4650 60  0001 C CNN
 F 3 "" H 9100 4650 60  0000 C CNN
 	1    9100 4650
@@
 F 0 "R1" V 8800 4650 50  0000 C CNN
 F 1 "20k" V 8900 4650 50  0000 C CNN
-F 2 "" H 8900 4650 60  0001 C CNN
+F 2 "pmod-wifi-esp32:SMD0603" H 8900 4650 60  0001 C CNN
 F 3 "" H 8900 4650 60  0000 C CNN
 	1    8900 4650
@@
 F 0 "C4" H 8900 3550 50  0000 L CNN
 F 1 "C" H 8900 3350 50  0000 L CNN
-F 2 "" H 8850 3450 60  0001 C CNN
+F 2 "pmod-wifi-esp32:SMD0603" H 8850 3450 60  0001 C CNN
 F 3 "" H 8850 3450 60  0000 C CNN
 	1    8850 3450
@@
 F 0 "L1" V 9400 3200 60  0000 C CNN
 F 1 "INDUCTOR" V 9200 3200 40  0000 C CNN
-F 2 "" H 9250 3200 60  0001 C CNN
+F 2 "pmod-wifi-esp32:SMD0603" H 9250 3200 60  0001 C CNN
 F 3 "" H 9250 3200 60  0000 C CNN
 	1    9250 3200
@@
 F 0 "C5" H 9700 3550 50  0000 L CNN
 F 1 "C" H 9700 3350 50  0000 L CNN
-F 2 "" H 9650 3450 60  0001 C CNN
+F 2 "pmod-wifi-esp32:SMD0603" H 9650 3450 60  0001 C CNN
 F 3 "" H 9650 3450 60  0000 C CNN
 	1    9650 3450
@@
 F 0 "C6" H 7400 4750 50  0000 R CNN
 F 1 "10pF" V 7550 4600 50  0000 R CNN
-F 2 "" H 7450 4650 60  0001 C CNN
+F 2 "pmod-wifi-esp32:SMD0603" H 7450 4650 60  0001 C CNN
 F 3 "" H 7450 4650 60  0000 C CNN
 	1    7450 4650
@@
 F 0 "C7" H 8100 4750 50  0000 L CNN
 F 1 "10pF" V 7950 4600 50  0000 R CNN
-F 2 "" H 8050 4650 60  0001 C CNN
+F 2 "pmod-wifi-esp32:SMD0603" H 8050 4650 60  0001 C CNN
 F 3 "" H 8050 4650 60  0000 C CNN
 	1    8050 4650
@@
 F 0 "A1" H 9862 3332 60  0000 R CNN
 F 1 "ANTENNA" H 9862 3241 40  0000 R CNN
-F 2 "" H 10050 3100 60  0001 C CNN
+F 2 "pmod-wifi-esp32:ANT_7488910245" H 10050 3100 60  0001 C CNN
 F 3 "" H 10050 3100 60  0000 C CNN
 	1    10050 3100
@@
 F 0 "C8" H 7050 2800 50  0000 R CNN
 F 1 "10nF" H 7050 2600 50  0000 R CNN
-F 2 "" H 7100 2700 60  0000 C CNN
+F 2 "pmod-wifi-esp32:SMD0603" H 7100 2700 60  0001 C CNN
 F 3 "" H 7100 2700 60  0000 C CNN
 	1    7100 2700
@@
 F 0 "L2" V 6850 2450 60  0000 C CNN
 F 1 "INDUCTOR" V 6650 2450 40  0000 C CNN
-F 2 "" H 6700 2450 60  0000 C CNN
+F 2 "pmod-wifi-esp32:SMD0603" H 6700 2450 60  0001 C CNN
 F 3 "" H 6700 2450 60  0000 C CNN
 	1    6700 2450
@@
 F 0 "C10" H 6350 2800 50  0000 L CNN
 F 1 "100nF" H 6350 2600 50  0000 L CNN
-F 2 "" H 6300 2700 60  0000 C CNN
+F 2 "pmod-wifi-esp32:SMD0603" H 6300 2700 60  0001 C CNN
 F 3 "" H 6300 2700 60  0000 C CNN
 	1    6300 2700
@@
 F 0 "C9" H 6050 2800 50  0000 L CNN
 F 1 "1uF" H 6050 2600 50  0000 L CNN
-F 2 "" H 6000 2700 60  0000 C CNN
+F 2 "pmod-wifi-esp32:SMD0603" H 6000 2700 60  0001 C CNN
 F 3 "" H 6000 2700 60  0000 C CNN
 	1    6000 2700
@@
 F 0 "R2" V 6400 3350 50  0000 C CNN
 F 1 "10k" V 6500 3350 50  0000 C CNN
-F 2 "" H 6500 3350 60  0000 C CNN
+F 2 "pmod-wifi-esp32:SMD0603" H 6500 3350 60  0001 C CNN
 F 3 "" H 6500 3350 60  0000 C CNN
 	1    6500 3350
@@
 F 0 "U1" H 4000 4400 60  0000 C CNN
 F 1 "ESP32" H 4000 2400 60  0000 C CNN
-F 2 "" H 4000 3500 60  0000 C CNN
+F 2 "pmod-wifi-esp32:QFN48-04" H 4000 3500 60  0001 C CNN
 F 3 "" H 4000 3500 60  0000 C CNN
 	2    4000 3350
@@
 F 0 "U2" H 4200 5950 60  0000 C CNN
 F 1 "M25P16-VME" H 4350 5050 60  0000 C CNN
-F 2 "" H 4000 5500 60  0000 C CNN
+F 2 "pmod-wifi-esp32:SOIC-8" H 4000 5500 60  0001 C CNN
 F 3 "" H 4000 5500 60  0000 C CNN
 	1    4000 5500
@@
 F 0 "C1" H 1650 4750 50  0000 L CNN
 F 1 "10uF" H 1650 4550 50  0000 L CNN
-F 2 "" H 1600 4650 60  0000 C CNN
+F 2 "pmod-wifi-esp32:SMD0805" H 1600 4650 60  0001 C CNN
 F 3 "" H 1600 4650 60  0000 C CNN
 	1    1600 4650
@@
 L pmod-wifi-esp32:VCC #PWR0123
 U 1 1 5F1E48E3
-P 1600 4400
-F 0 "#PWR0123" H 1600 4360 30  0001 C CNN
-F 1 "VCC" H 1609 4538 30  0000 C CNN
-F 2 "" H 1600 4400 60  0000 C CNN
-F 3 "" H 1600 4400 60  0000 C CNN
-	1    1600 4400
+P 1600 4350
+F 0 "#PWR0123" H 1600 4310 30  0001 C CNN
+F 1 "VCC" H 1609 4488 30  0000 C CNN
+F 2 "" H 1600 4350 60  0000 C CNN
+F 3 "" H 1600 4350 60  0000 C CNN
+	1    1600 4350
 	1    0    0    -1
 $EndComp
@@
 Wire Wire Line
 	1600 4900 1600 4850
-Wire Wire Line
-	1600 4450 1600 4400
 Text GLabel 2050 3300 2    50   Output ~ 0
 PMOD_RST
@@
 F 0 "C11" H 2700 5600 50  0000 L CNN
 F 1 "100nF" H 2700 5400 50  0000 L CNN
-F 2 "" H 2650 5500 60  0000 C CNN
+F 2 "pmod-wifi-esp32:SMD0603" H 2650 5500 60  0001 C CNN
 F 3 "" H 2650 5500 60  0000 C CNN
 	1    2650 5500
@@
 F 0 "TP1" H 3250 3850 40  0000 L CNN
 F 1 "CONN_1" H 3200 3905 30  0001 C CNN
-F 2 "" H 3200 3850 60  0000 C CNN
+F 2 "pmod-wifi-esp32:TP_SMD" H 3200 3850 60  0001 C CNN
 F 3 "" H 3200 3850 60  0000 C CNN
 	1    3200 3850
@@
 F 0 "TP2" H 3250 3950 40  0000 L CNN
 F 1 "CONN_1" H 3200 4005 30  0001 C CNN
-F 2 "" H 3200 3950 60  0000 C CNN
+F 2 "pmod-wifi-esp32:TP_SMD" H 3200 3950 60  0001 C CNN
 F 3 "" H 3200 3950 60  0000 C CNN
 	1    3200 3950
@@
 F 0 "TP3" H 3250 4050 40  0000 L CNN
 F 1 "CONN_1" H 3200 4105 30  0001 C CNN
-F 2 "" H 3200 4050 60  0000 C CNN
+F 2 "pmod-wifi-esp32:TP_SMD" H 3200 4050 60  0001 C CNN
 F 3 "" H 3200 4050 60  0000 C CNN
 	1    3200 4050
@@
 F 0 "TP4" H 3250 4150 40  0000 L CNN
 F 1 "CONN_1" H 3200 4205 30  0001 C CNN
-F 2 "" H 3200 4150 60  0000 C CNN
+F 2 "pmod-wifi-esp32:TP_SMD" H 3200 4150 60  0001 C CNN
 F 3 "" H 3200 4150 60  0000 C CNN
 	1    3200 4150
@@
 Wire Wire Line
 	3450 4150 3350 4150
+$Comp
+L pmod-wifi-esp32:INDUCTOR FB1
+U 1 1 5F17A32A
+P 2050 4400
+F 0 "FB1" V 2150 4400 40  0000 C CNN
+F 1 "FB120" V 2000 4400 40  0000 C CNN
+F 2 "pmod-wifi-esp32:SMD0603" H 2050 4400 60  0001 C CNN
+F 3 "" H 2050 4400 60  0000 C CNN
+	1    2050 4400
+	0    -1   -1   0
+$EndComp
+Wire Wire Line
+	1600 4400 1750 4400
+Wire Wire Line
+	1600 4350 1600 4400
+Connection ~ 1600 4400
+Wire Wire Line
+	1600 4400 1600 4450
+$Comp
+L pmod-wifi-esp32:+3.3V #PWR0127
+U 1 1 5F183E53
+P 2450 4350
+F 0 "#PWR0127" H 2450 4310 30  0001 C CNN
+F 1 "+3.3V" H 2459 4488 30  0000 C CNN
+F 2 "" H 2450 4350 60  0000 C CNN
+F 3 "" H 2450 4350 60  0000 C CNN
+	1    2450 4350
+	1    0    0    -1
+$EndComp
+Wire Wire Line
+	2450 4350 2450 4400
+Wire Wire Line
+	2450 4400 2350 4400
+$Comp
+L pmod-wifi-esp32:C C12
+U 1 1 5F17B079
+P 6400 4650
+F 0 "C12" H 6530 4696 50  0000 L CNN
+F 1 "100nF" H 6530 4605 50  0000 L CNN
+F 2 "pmod-wifi-esp32:SMD0603" H 6400 4650 60  0001 C CNN
+F 3 "" H 6400 4650 60  0000 C CNN
+	1    6400 4650
+	1    0    0    -1
+$EndComp
+$Comp
+L pmod-wifi-esp32:+3.3V #PWR0128
+U 1 1 5F17B19D
+P 6400 4400
+F 0 "#PWR0128" H 6400 4360 30  0001 C CNN
+F 1 "+3.3V" H 6409 4538 30  0000 C CNN
+F 2 "" H 6400 4400 60  0000 C CNN
+F 3 "" H 6400 4400 60  0000 C CNN
+	1    6400 4400
+	1    0    0    -1
+$EndComp
+$Comp
+L pmod-wifi-esp32:GND #PWR0129
+U 1 1 5F17B217
+P 6400 4900
+F 0 "#PWR0129" H 6400 4900 30  0001 C CNN
+F 1 "GND" H 6400 4830 30  0001 C CNN
+F 2 "" H 6400 4900 60  0000 C CNN
+F 3 "" H 6400 4900 60  0000 C CNN
+	1    6400 4900
+	1    0    0    -1
+$EndComp
+Wire Wire Line
+	6400 4900 6400 4850
+Wire Wire Line
+	6400 4450 6400 4400
 $EndSCHEMATC

Commit message: = UPD: Fix bug of flash memory ios ; add a signal to control "boot" pin from pmod
Connections:
- net PMOD_BOOT: now reaches P1.9 (IO7)
- net PMOD_BOOT: now also U1.23 (GPIO0)
- net FL_D0 renamed FL_SDI
- net FL_SDI: now also U1.33 (SD_DAT1); no longer U1.32 (SD_DAT0)
- net FL_D1 renamed FL_SDO
- net FL_SDO: now also U1.32 (SD_DAT0); no longer U1.33 (SD_DAT1)
- net FL_D2 renamed FL_SHD
- net FL_SHD: now also U2.7 (IO3_HOLD); no longer U2.3 (IO2_WP)
- net FL_D3 renamed FL_SWP
- net FL_SWP: now also U2.3 (IO2_WP); no longer U2.7 (IO3_HOLD)
- no-connect marks 22 -> 20
Changed lines of the file:
@@
 Sheet 1 1
 Title "PMOD Wifi ESP32"
-Date "2020-07-20"
-Rev "1"
+Date "2020-08-28"
+Rev "2"
 Comp "Agilack"
 Comment1 "License: CC-by-SA 2.0"
@@
 	4550 2850 4650 2850
 Text GLabel 4650 2850 2    45   BiDi ~ 0
-FL_D0
+FL_SDO
 Wire Wire Line
 	4650 2750 4550 2750
 Text GLabel 4650 2950 2    45   BiDi ~ 0
-FL_D1
+FL_SDI
 Text GLabel 4650 3050 2    45   BiDi ~ 0
-FL_D2
+FL_SHD
 Text GLabel 4650 3150 2    45   BiDi ~ 0
-FL_D3
+FL_SWP
 Wire Wire Line
 	4650 3150 4550 3150
@@
 Wire Wire Line
 	1550 3750 1550 3800
-NoConn ~ 1950 3400
 NoConn ~ 1950 3500
 Text GLabel 4650 3950 2    45   Input ~ 0
@@
 NoConn ~ 3450 2950
 NoConn ~ 3450 3050
-NoConn ~ 3450 3150
 NoConn ~ 3450 3250
 $Comp
@@
 	3500 5350 3400 5350
 Text GLabel 4550 5250 2    50   BiDi ~ 0
-FL_D0
+FL_SDI
 Text GLabel 4550 5400 2    50   BiDi ~ 0
-FL_D1
+FL_SDO
 Text GLabel 4550 5600 2    50   BiDi ~ 0
-FL_D2
+FL_SWP
 Text GLabel 4550 5750 2    50   BiDi ~ 0
-FL_D3
+FL_SHD
 Wire Wire Line
 	4550 5750 4450 5750
@@
 Wire Wire Line
 	6400 4450 6400 4400
+Text GLabel 3350 3150 0    45   Input ~ 0
+PMOD_BOOT
+Wire Wire Line
+	3350 3150 3450 3150
+Text GLabel 2050 3400 2    45   Output ~ 0
+PMOD_BOOT
+Wire Wire Line
+	2050 3400 1950 3400
 $EndSCHEMATC
